File: remote-control/kumanda_pcb/kumanda/kumanda.sch (KiCad schematic (older format))
At the start: 38 parts, among them J1 USB_A, J2 Conn_01x04, J3 RJ45, J4 Conn_01x06, J5 Screw_Terminal_01x02, U1 MEGA_PRO_EMBED_CH340G___ATMEG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

Commit message: PCB design finished.
Parts:
- Bluetooth1: renamed from J2; footprint Connector_Molex:Molex_KK-254_AE-6410-04A_1x04_P2.54mm_Vertical -> Connector_JST:JST_XH_B4B-XH-A_1x04_P2.50mm_Vertical
- DHT1, POT1, POT2, Switch1, Switch2, VIB1, VIB2: footprint Connector_Molex:Molex_KK-254_AE-6410-03A_1x03_P2.54mm_Vertical -> Connector_JST:JST_XH_B3B-XH-A_1x03_P2.50mm_Vertical
- Joy1, Joy2: footprint Connector_Molex:Molex_KK-254_AE-6410-05A_1x05_P2.54mm_Vertical -> Connector_JST:JST_XH_B5B-XH-A_1x05_P2.50mm_Vertical
- OLED_I2C1: footprint Connector_Molex:Molex_KK-254_AE-6410-04A_1x04_P2.54mm_Vertical -> Connector_JST:JST_XH_B4B-XH-A_1x04_P2.50mm_Vertical
- U1: footprint MODULE_MEGA_PRO_EMBED_CH340G_git:_ATMEGA2560 -> MODULE_MEGA_PRO_EMBED_CH340G_:_ATMEGA2560; symbol MEGA_PRO_EMBED_CH340G___ATMEGA2560-git:MEGA_PRO_EMBED_CH340G___ATMEGA2560 -> kumanda-rescue:MEGA_PRO_EMBED_CH340G___ATMEGA2560-MEGA_PRO_EMBED_CH340G___ATMEGA2560-git
- renumbered J4 to AV_conv1, J3 to RJ45, J5 to screw_term1
Connections:
- net 5v is gone; now on net VBUS: USB_kod1.5 (Pin_5)
- net RX: now also U1.RX
- net TX: now also U1.TX
Changed lines of the file:
@@
 F 0 "VIB1" H 2980 5892 50  0000 L CNN
 F 1 "Conn_01x03" H 2980 5801 50  0000 L CNN
-F 2 "Connector_Molex:Molex_KK-254_AE-6410-03A_1x03_P2.54mm_Vertical" H 2900 5850 50  0001 C CNN
+F 2 "Connector_JST:JST_XH_B3B-XH-A_1x03_P2.50mm_Vertical" H 2900 5850 50  0001 C CNN
 F 3 "~" H 2900 5850 50  0001 C CNN
 	1    2900 5850
@@
 F 0 "POT1" H 2980 3792 50  0000 L CNN
 F 1 "Conn_01x03" H 2980 3701 50  0000 L CNN
-F 2 "Connector_Molex:Molex_KK-254_AE-6410-03A_1x03_P2.54mm_Vertical" H 2900 3750 50  0001 C CNN
+F 2 "Connector_JST:JST_XH_B3B-XH-A_1x03_P2.50mm_Vertical" H 2900 3750 50  0001 C CNN
 F 3 "~" H 2900 3750 50  0001 C CNN
 	1    2900 3750
@@
 F 0 "POT2" H 9630 3892 50  0000 L CNN
 F 1 "Conn_01x03" H 9630 3801 50  0000 L CNN
-F 2 "Connector_Molex:Molex_KK-254_AE-6410-03A_1x03_P2.54mm_Vertical" H 9550 3850 50  0001 C CNN
+F 2 "Connector_JST:JST_XH_B3B-XH-A_1x03_P2.50mm_Vertical" H 9550 3850 50  0001 C CNN
 F 3 "~" H 9550 3850 50  0001 C CNN
 	1    9550 3850
@@
 F 0 "DHT1" H 2980 5192 50  0000 L CNN
 F 1 "Conn_01x03" H 2980 5101 50  0000 L CNN
-F 2 "Connector_Molex:Molex_KK-254_AE-6410-03A_1x03_P2.54mm_Vertical" H 2900 5150 50  0001 C CNN
+F 2 "Connector_JST:JST_XH_B3B-XH-A_1x03_P2.50mm_Vertical" H 2900 5150 50  0001 C CNN
 F 3 "~" H 2900 5150 50  0001 C CNN
 	1    2900 5150
@@
 F 0 "OLED_I2C1" H 4830 5792 50  0000 L CNN
 F 1 "Conn_01x04" H 4830 5701 50  0000 L CNN
-F 2 "Connector_Molex:Molex_KK-254_AE-6410-04A_1x04_P2.54mm_Vertical" H 4750 5800 50  0001 C CNN
+F 2 "Connector_JST:JST_XH_B4B-XH-A_1x04_P2.50mm_Vertical" H 4750 5800 50  0001 C CNN
 F 3 "~" H 4750 5800 50  0001 C CNN
 	1    4750 5800
@@
 F 0 "VIB2" H 9630 5142 50  0000 L CNN
 F 1 "Conn_01x03" H 9630 5051 50  0000 L CNN
-F 2 "Connector_Molex:Molex_KK-254_AE-6410-03A_1x03_P2.54mm_Vertical" H 9550 5100 50  0001 C CNN
+F 2 "Connector_JST:JST_XH_B3B-XH-A_1x03_P2.50mm_Vertical" H 9550 5100 50  0001 C CNN
 F 3 "~" H 9550 5100 50  0001 C CNN
 	1    9550 5100
@@
 $EndComp
 $Comp
-L Connector:RJ45 J3
+L Connector:RJ45 RJ45
 U 1 1 60C7E37E
 P 6200 2700
-F 0 "J3" H 6257 3367 50  0000 C CNN
+F 0 "RJ45" H 6257 3367 50  0000 C CNN
 F 1 "RJ45" H 6257 3276 50  0000 C CNN
 F 2 "Connector_RJ:RJ45_Ninigi_GE" V 6200 2725 50  0001 C CNN
@@
 F 0 "Joy1" H 2980 4392 50  0000 L CNN
 F 1 "Conn_01x05" H 2980 4301 50  0000 L CNN
-F 2 "Connector_Molex:Molex_KK-254_AE-6410-05A_1x05_P2.54mm_Vertical" H 2900 4350 50  0001 C CNN
+F 2 "Connector_JST:JST_XH_B5B-XH-A_1x05_P2.50mm_Vertical" H 2900 4350 50  0001 C CNN
 F 3 "~" H 2900 4350 50  0001 C CNN
 	1    2900 4350
@@
 F 0 "Joy2" H 9630 4492 50  0000 L CNN
 F 1 "Conn_01x05" H 9630 4401 50  0000 L CNN
-F 2 "Connector_Molex:Molex_KK-254_AE-6410-05A_1x05_P2.54mm_Vertical" H 9550 4450 50  0001 C CNN
+F 2 "Connector_JST:JST_XH_B5B-XH-A_1x05_P2.50mm_Vertical" H 9550 4450 50  0001 C CNN
 F 3 "~" H 9550 4450 50  0001 C CNN
 	1    9550 4450
@@
 F 0 "Switch1" H 3030 3092 50  0000 L CNN
 F 1 "Conn_01x03" H 3030 3001 50  0000 L CNN
-F 2 "Connector_Molex:Molex_KK-254_AE-6410-03A_1x03_P2.54mm_Vertical" H 2950 3050 50  0001 C CNN
+F 2 "Connector_JST:JST_XH_B3B-XH-A_1x03_P2.50mm_Vertical" H 2950 3050 50  0001 C CNN
 F 3 "~" H 2950 3050 50  0001 C CNN
 	1    2950 3050
@@
 F 0 "Switch2" H 9630 3492 50  0000 L CNN
 F 1 "Conn_01x03" H 9630 3401 50  0000 L CNN
-F 2 "Connector_Molex:Molex_KK-254_AE-6410-03A_1x03_P2.54mm_Vertical" H 9550 3450 50  0001 C CNN
+F 2 "Connector_JST:JST_XH_B3B-XH-A_1x03_P2.50mm_Vertical" H 9550 3450 50  0001 C CNN
 F 3 "~" H 9550 3450 50  0001 C CNN
 	1    9550 3450
@@
 Connection ~ 9250 4350
 $Comp
-L Connector_Generic:Conn_01x04 J2
+L Connector_Generic:Conn_01x04 Bluetooth1
 U 1 1 60D1844F
 P 8800 5800
-F 0 "J2" V 8672 5980 50  0000 L CNN
+F 0 "Bluetooth1" V 8672 5980 50  0000 L CNN
 F 1 "Conn_01x04" V 8763 5980 50  0000 L CNN
-F 2 "Connector_Molex:Molex_KK-254_AE-6410-04A_1x04_P2.54mm_Vertical" H 8800 5800 50  0001 C CNN
+F 2 "Connector_JST:JST_XH_B4B-XH-A_1x04_P2.50mm_Vertical" H 8800 5800 50  0001 C CNN
 F 3 "~" H 8800 5800 50  0001 C CNN
 	1    8800 5800
@@
 GND
 $Comp
-L Connector_Generic:Conn_01x06 J4
+L Connector_Generic:Conn_01x06 AV_conv1
 U 1 1 60CAFA0F
 P 1850 6800
-F 0 "J4" H 1930 6792 50  0000 L CNN
+F 0 "AV_conv1" H 1930 6792 50  0000 L CNN
 F 1 "Conn_01x06" H 1930 6701 50  0000 L CNN
 F 2 "analog_cam:Analog-cam" H 1850 6800 50  0001 C CNN
@@
 	6150 3550 3300 3550
 $Comp
-L MEGA_PRO_EMBED_CH340G___ATMEGA2560-git:MEGA_PRO_EMBED_CH340G___ATMEGA2560 U1
+L kumanda-rescue:MEGA_PRO_EMBED_CH340G___ATMEGA2560-MEGA_PRO_EMBED_CH340G___ATMEGA2560-git U1
 U 1 1 60C9CA00
 P 6200 4300
 F 0 "U1" V 6246 6830 50  0000 L CNN
 F 1 "MEGA_PRO_EMBED_CH340G___ATMEGA2560" V 6155 6830 50  0000 L CNN
-F 2 "MODULE_MEGA_PRO_EMBED_CH340G_git:_ATMEGA2560" H 6200 4300 50  0001 L BNN
+F 2 "MODULE_MEGA_PRO_EMBED_CH340G_:_ATMEGA2560" H 6200 4300 50  0001 L BNN
 F 3 "" H 6200 4300 50  0001 L BNN
 F 4 "12/May/2017" H 6200 4300 50  0001 L BNN "PARTREV"
@@
 3.3V
 $Comp
-L Connector:Screw_Terminal_01x02 J5
+L Connector:Screw_Terminal_01x02 screw_term1
 U 1 1 6122B52B
 P 1125 3775
-F 0 "J5" H 1043 3450 50  0000 C CNN
+F 0 "screw_term1" H 1043 3450 50  0000 C CNN
 F 1 "Screw_Terminal_01x02" H 1043 3541 50  0000 C CNN
 F 2 "TerminalBlock_Phoenix:TerminalBlock_Phoenix_PT-1,5-2-3.5-H_1x02_P3.50mm_Horizontal" H 1125 3775 50  0001 C CNN
@@
 Text GLabel 1125 5100 0    50   Input ~ 0
 GND
-Text GLabel 1125 5200 0    50   Input ~ 0
-5v
 Text GLabel 1125 5300 0    50   Input ~ 0
 DTR
 Text GLabel 4700 5000 3    50   Input ~ 0
 DTR
+Text GLabel 1125 5200 0    50   Input ~ 0
+VCC
+Text GLabel 4400 3600 1    50   Input ~ 0
+RX
+Text GLabel 4300 3600 1    50   Input ~ 0
+TX
 $EndSCHEMATC
